File: USBAudioInterface/audiointerf.kicad_sch (KiCad schematic)
At the start: 47 parts, among them IC1 REG103GA-2.5, IC2 PCM2900CDB, J1 USB_B, J2 AudioJack4, J3 AudioJack4, SW1 SW_Push, SW2 SW_Push, SW3 SW_Push, U1 OPA1622, U2 OPA1622, Y1 Crystal

Commit message: Add files via upload
Parts:
- removed IC1: REG103GA-2.5, SOT127P706X180-6N, symbol REG103GA-2.5:REG103GA-2.5
- removed J2, J3: AudioJack4, symbol Connector:AudioJack4
- added IC1: REG103GA-A, Package_TO_SOT_SMD:SOT-223-6, symbol REG103GA-A:REG103GA-A
- added J2: AudioJack3, Connector_Audio:Jack_6.35mm_Neutrik_NJ3FD-V_Vertical, symbol Connector:AudioJack3
- added J3: AudioJack3, Connector_Audio:Jack_3.5mm_CUI_SJ-3523-SMT_Horizontal, symbol Connector:AudioJack3
- C1, C10, C13, C14, C17, C18, C2, C7, C8, C9: footprint (none) -> Capacitor_Tantalum_SMD:CP_EIA-2012-15_AVX-P
- C11, C12, C3, C4, C5, C6: footprint (none) -> Capacitor_THT:CP_Radial_D5.0mm_P2.50mm
- C15: renamed from C16; footprint (none) -> Capacitor_Tantalum_SMD:CP_EIA-2012-15_AVX-P
- C16: renamed from C15; footprint (none) -> Capacitor_Tantalum_SMD:CP_EIA-2012-15_AVX-P
- D1: footprint (none) -> Diode_SMD:D_2114_3652Metric
- IC2: footprint SOP65P780X200-28N -> Package_SO:SSOP-28_5.3x10.2mm_P0.65mm
- J1: footprint (none) -> Connector_USB:USB_B_Lumberg_2411_02_Horizontal
- R1, R10, R11, R12, R15, R16, R2, R3, R4, R5, R6, R7, R8, R9: footprint (none) -> Resistor_SMD:R_0603_1608Metric
- R13: renamed from R14; footprint (none) -> Resistor_SMD:R_0603_1608Metric
- R14: renamed from R13; footprint (none) -> Resistor_SMD:R_0603_1608Metric
- RV1: footprint (none) -> Potentiometer_THT:Potentiometer_Alpha_RD902F-40-00D_Dual_Vertical
- SW1, SW2, SW3: footprint (none) -> Button_Switch_THT:SW_CW_GPTS203211B
- Y1: footprint (none) -> Crystal:Crystal_DS10_D1.0mm_L4.3mm_Horizontal
- renumbered U2 to U1, U1 to U2
Connections:
- net GND: now also IC1.3 (GND), IC1.6 (GND_1), J2.S, J3.S
- net VINR: now reaches C4.1, IC2.13 (VINR)
- net at C4.2: now also J2.R
- net ENABLE: now reaches IC2.28 (~{SSPND}), R4.1, R5.1, R6.1
- net ENABLE: now also IC1.5 (ENABLE)
- net VINL: now reaches C3.1, IC2.12 (VINL)
- net at C3.2: now also J2.T
- net at C1.1, J1.1 (VBUS), R3.1: now also IC1.1 (VIN)
- net VCCCI: now reaches D1.2 (A), R1.1
- net VCCCI: now also IC1.2 (VOUT)
- net at R1.2, R2.1: now also IC1.4 (NR/ADJUST)
- net at C17.2: now also J3.R
- net at C18.2: now also J3.T
- net VOUTL: now reaches IC2.16 (VOUTL), RV1.1
- net VOUTR: now reaches IC2.15 (VOUTR), RV1.4
- no-connect marks 0 -> 2
Other:
- moved on the sheet: C1, C15, C18, C3, C4, C6, R1, R13, R16, R2, RV1, U1B
