File: USBAudioInterface/audiointerf.kicad_pcb (KiCad board)
At the start: 4 copper layers, 47 parts, among them IC1 REG103GA-A, IC2 PCM2900CDB, J1 USB_B, J2 AudioJack3, J3 AudioJack3, SW1 SW_Push, SW2 SW_Push, SW3 SW_Push, U1 OPA1622, U2 OPA1622, Y1 Crystal

Commit message: updates files
Parts:
- added REF**: MountingHole_2.2mm_M2, MountingHole:MountingHole_2.2mm_M2, F.Cu at (43.9, 59.9)
- added REF**: MountingHole_2.2mm_M2, MountingHole:MountingHole_2.2mm_M2, F.Cu at (105.9, 59.7)
- added REF**: MountingHole_2.2mm_M2, MountingHole:MountingHole_2.2mm_M2, F.Cu at (44.0, 134.0)
- moved C17 94.3 mm to (78.6, 124.5)
- moved C18 93.4 mm to (89.8, 124.5)
- moved R15 91.8 mm to (75.7, 123.8), turned to -90 degrees
- moved R16 91.3 mm to (86.9, 123.8), turned to -90 degrees
- moved J3 88.1 mm to (99.3, 127.3), turned to 180 degrees
- moved C16 87.8 mm to (72.6, 120.3), turned to -90 degrees
- moved R14 86.1 mm to (74.4, 120.2), turned to -90 degrees
- moved U2 81.6 mm to (79.0, 120.1), turned to 180 degrees
- moved C15 78.2 mm to (84.1, 120.1), turned to -90 degrees
- moved R13 75.1 mm to (85.9, 120.1), turned to -90 degrees
- moved R12 70.8 mm to (81.7, 116.6), turned to 180 degrees
- moved U1 70.2 mm to (89.9, 120.1), turned to 180 degrees
- moved R11 59.8 mm to (91.4, 116.6), turned to 180 degrees
- moved C12 28.8 mm to (85.9, 113.1), turned to -90 degrees
- moved C11 17.1 mm to (95.5, 113.1), turned to -90 degrees
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Connections:
- R13 pad 1: Net-(C15-Pad2) -> Net-(C15-Pad1)
- R13 pad 2: Net-(C15-Pad1) -> Net-(C15-Pad2)
Routing:
- net GND: track 103.5 -> 301.3 mm, vias 11 -> 13
- net Net-(C10-Pad1): track 11.0 -> 31.9 mm, vias 1 -> 0
- net Net-(C17-Pad2): track 0.00 -> 20.2 mm, vias 0 -> 2
- net Net-(C18-Pad2): track 0.00 -> 16.3 mm, vias 0 -> 2
- net Net-(C1-Pad1): track 8.30 -> 24.0 mm
- net /VOUTL: track 0.00 -> 11.3 mm
- net Net-(C16-Pad1): track 0.00 -> 11.3 mm
- net Net-(C11-Pad1): track 0.00 -> 9.90 mm
- net Net-(C15-Pad1): track 0.00 -> 9.75 mm
- net /VCCCI: track 5.56 -> 15.1 mm
- net Net-(C12-Pad1): track 0.00 -> 8.94 mm
- net /VOUTR: track 0.00 -> 8.55 mm
- net Net-(C16-Pad2): track 0.00 -> 8.15 mm
- net Net-(C15-Pad2): track 0.00 -> 7.53 mm
- net Net-(C3-Pad2): track 8.06 -> 15.4 mm
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Other:
- board outline added: 70 x 82 mm
