File: pdb/pdb.kicad_sch (KiCad schematic)
At the start: 11 parts, among them J1 Conn_01x02, U1 INA169, U2 LM7812_TO220, U3 NCP1117-5.0_TO252

Commit message: updated circuit and picture
Connections:
- net GND: now also J1.1 (Pin_1); no longer J1.2 (Pin_2)
- net at RS1.1, RS2.1, U1.3 (+)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: now also J1.2 (Pin_2); no longer J1.1 (Pin_1)
Changed lines of the file:
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@@
-    (stroke (width 0) (type default) (color 0 0 0 0))
-  )
-  (wire (pts (xy 26.67 97.79) (xy 38.1 97.79))
     (stroke (width 0) (type default) (color 0 0 0 0))
   )
@@
   )
   (wire (pts (xy 38.1 69.85) (xy 62.23 69.85))
+    (stroke (width 0) (type default) (color 0 0 0 0))
+  )
+  (wire (pts (xy 27.94 97.79) (xy 26.67 97.79))
     (stroke (width 0) (type default) (color 0 0 0 0))
   )
@@
     (stroke (width 0) (type default) (color 0 0 0 0))
   )
-  (wire (pts (xy 38.1 97.79) (xy 38.1 69.85))
+  (wire (pts (xy 38.1 69.85) (xy 38.1 100.33))
     (stroke (width 0) (type default) (color 0 0 0 0))
   )
@@
     (stroke (width 0) (type default) (color 0 0 0 0))
   )
+  (wire (pts (xy 27.94 95.25) (xy 27.94 97.79))
+    (stroke (width 0) (type default) (color 0 0 0 0))
+  )
   (wire (pts (xy 76.2 53.34) (xy 76.2 58.42))
     (stroke (width 0) (type default) (color 0 0 0 0))
@@
     (stroke (width 0) (type default) (color 0 0 0 0))
   )
-  (wire (pts (xy 26.67 100.33) (xy 26.67 102.87))
-    (stroke (width 0) (type default) (color 0 0 0 0))
-  )
   (wire (pts (xy 129.54 58.42) (xy 129.54 110.49))
     (stroke (width 0) (type default) (color 0 0 0 0))
   )
   (wire (pts (xy 72.39 64.77) (xy 76.2 64.77))
+    (stroke (width 0) (type default) (color 0 0 0 0))
+  )
+  (wire (pts (xy 38.1 100.33) (xy 26.67 100.33))
     (stroke (width 0) (type default) (color 0 0 0 0))
   )
@@
     )
   )
-  (symbol (lib_id "power:GND") (at 26.67 102.87 0) (unit 1)
+  (symbol (lib_id "power:GND") (at 27.94 95.25 180) (unit 1)
     (in_bom yes) (on_board yes) (fields_autoplaced)
-    (property "Reference" "#PWR01" (id 0) (at 26.67 109.22 0)
+    (property "Reference" "#PWR01" (id 0) (at 27.94 88.9 0)
       (effects (font (size 1.27 1.27)) hide)
     )
-    (property "Value" "GND" (id 1) (at 26.67 107.95 0))
-    (property "Footprint" "" (id 2) (at 26.67 102.87 0)
+    (property "Value" "GND" (id 1) (at 27.94 90.17 0))
+    (property "Footprint" "" (id 2) (at 27.94 95.25 0)
       (effects (font (size 1.27 1.27)) hide)
     )
-    (property "Datasheet" "" (id 3) (at 26.67 102.87 0)
+    (property "Datasheet" "" (id 3) (at 27.94 95.25 0)
       (effects (font (size 1.27 1.27)) hide)
     )
